Commit message: a

File: install/my_robot_description/share/my_robot_description/urdf/common_properties.xacro (robot description, xacro)
@@ -5,5 +5,5 @@
             <visual>
                 <geometry>
-                    <cylinder radius="${wheel_radius}" length="${wheel_lenght}"/>
+                    <cylinder radius="${wheel_radius}" length="${wheel_length}"/>
                 </geometry>
                 <origin xyz="0 0 0" rpy="1.5708 0 0"/> <!-- pi/2 ≈ 1.5708 -->
@@ -12,9 +12,9 @@
             <collision>
                 <geometry>
-                    <cylinder radius="${wheel_radius}" length="${wheel_lenght}"/>
+                    <cylinder radius="${wheel_radius}" length="${wheel_length}"/>
                 </geometry>
                 <origin xyz="0 0 0" rpy="1.5708 0 0"/> <!-- pi/2 ≈ 1.5708 -->
             </collision>
-            <xacro:wheel_inertia m = "1.0" r = "${wheel_radius}" h = "${wheel_lenght}" xyz="0 0 0" rpy="1.5708 0 0"/>
+            <xacro:wheel_inertia m = "1.0" r = "${wheel_radius}" h = "${wheel_length}" xyz="0 0 0" rpy="1.5708 0 0"/>
         </link>
     </xacro:macro>
@@ -33,5 +33,5 @@
             <inertia ixx = "${(m/12) * (l*l+h*h)}" ixy = "0" ixz = "0"
             iyy = "${(m/12) * (l*l+h*h)}" iyz = "0"
-            izz = "${(m*r*r)/2}"/>
+            izz = "${(m/12) * (l*l+h*h)}"/>
         </inertial>
     </xacro:macro>
@@ -45,12 +45,13 @@
         </inertial>
     </xacro:macro>
-    <xacro:macro name = "sphere_inertia" params = "m r xyz rpy">
-        <inertia>
-            <origin xyz = "${xyz}" rpy = "${rpy}" />
-            <mass value = "${m}" />
-            <inertia ixx = "(2*m*r*r)/5" ixy = "0" ixz = "0"
-            iyy= "(2*m*r*r)/5" iyz = "0"
-            izz = "(2*m*r*r)/5"/>
-        </inertia>
-    </xacro:macro>
+    <xacro:macro name="sphere_inertia" params="m r xyz rpy">
+    <inertial>
+        <origin xyz="${xyz}" rpy="${rpy}"/>
+        <mass value="${m}"/>
+        <inertia
+            ixx="${(2 * m * r * r) / 5.0}" ixy="0" ixz="0"
+            iyy="${(2 * m * r * r) / 5.0}" iyz="0"
+            izz="${(2 * m * r * r) / 5.0}"/>
+    </inertial>
+</xacro:macro>
 </robot>

File: install/my_robot_description/share/my_robot_description/urdf/mobile_base.xacro (robot description, xacro)
@@ -5,5 +5,5 @@
     <xacro:property name="base_height" value="0.2" />
     <xacro:property name="wheel_radius" value="0.1" />
-    <xacro:property name="wheel_lenght" value="0.05" />
+    <xacro:property name="wheel_length" value="0.05" />
     <xacro:property name="sphere_radius" value="0.05" />
     <material name="blue">
@@ -28,10 +28,10 @@
             <origin xyz="0 0 ${base_height / 2.0}" rpy="0 0 0"/>
         </collision>
-        <xacro:box_inertia  m="5.0" l = "${base_length}" w="${base_width}" h = "${base_height}" xyz="0 0 ${base_height / 2.0}" rpy="0 0 0" />
+        <xacro:box_inertia m="5.0" l="${base_length}" w="${base_width}" h="${base_height}" xyz="0 0 ${base_height / 2.0}" rpy="0 0 0"/>
     </link>
     <link name="caster_wheel_link">
         <visual>
             <geometry>
-                <sphere radius="${wheel_radius / 2 }"/>
+                <sphere radius="${wheel_radius / 2.0}"/>
             </geometry>
             <origin xyz="0 0 0" rpy="0 0 0"/>
@@ -40,9 +40,9 @@
         <collision>
             <geometry>
-                <sphere radius="${wheel_radius / 2 }"/>
+                <sphere radius="${wheel_radius / 2.0}"/>
             </geometry>
             <origin xyz="0 0 0" rpy="0 0 0"/>
         </collision>
-        <xacro:sphere_inertia m = "1.0" r = "${wheel_radius / 2}" xyz="0 0 0" rpy="0 0 0"/>
+        <xacro:sphere_inertia m="1.0" r="${wheel_radius / 2.0}" xyz="0 0 0" rpy="0 0 0"/>
     </link>
     <xacro:wheel_link prefix="right" />

File: install/my_robot_description/share/my_robot_description/urdf/my_robot.urdf.xacro (robot description, xacro)
@@ -2,4 +2,4 @@
 <robot name="my_robot" xmlns:xacro="http://www.ros.org/wiki/xacro">
     <xacro:include filename = "/home/tayya/robot_ws/src/my_robot_description/urdf/common_properties.xacro" />
-    <xacro:include filename ="/home/tayya/robot_ws/src/my_robot_description/urdf/common_properties.xacro"/>
+    <xacro:include filename ="/home/tayya/robot_ws/src/my_robot_description/urdf/mobile_base.xacro"/>
 </robot>

Commit message: beforo_final

File: install/my_robot_description/share/my_robot_description/urdf/common_properties.xacro (robot description, xacro)
@@ -1,22 +1,4 @@
 <?xml version ="1.0"?>
 <robot xmlns:xacro="http://www.ros.org/wiki/xacro">
-    <xacro:macro name="wheel_link" params="prefix">
-        <link name="${prefix}_wheel_link">
-            <visual>
-                <geometry>
-                    <cylinder radius="${wheel_radius}" length="${wheel_length}"/>
-                </geometry>
-                <origin xyz="0 0 0" rpy="1.5708 0 0"/> <!-- pi/2 ≈ 1.5708 -->
-                <material name="grey"/>
-            </visual>
-            <collision>
-                <geometry>
-                    <cylinder radius="${wheel_radius}" length="${wheel_length}"/>
-                </geometry>
-                <origin xyz="0 0 0" rpy="1.5708 0 0"/> <!-- pi/2 ≈ 1.5708 -->
-            </collision>
-            <xacro:wheel_inertia m = "1.0" r = "${wheel_radius}" h = "${wheel_length}" xyz="0 0 0" rpy="1.5708 0 0"/>
-        </link>
-    </xacro:macro>
     <xacro:macro name="wheel_joint" params="prefix x y z">
         <joint name="${prefix}_wheel_joint" type="continuous">

File: install/my_robot_description/share/my_robot_description/urdf/mobile_base.xacro (robot description, xacro)
@@ -28,6 +28,24 @@
             <origin xyz="0 0 ${base_height / 2.0}" rpy="0 0 0"/>
         </collision>
-        <xacro:box_inertia m="5.0" l="${base_length}" w="${base_width}" h="${base_height}" xyz="0 0 ${base_height / 2.0}" rpy="0 0 0"/>
+        <xacro:box_inertia m="5.0" l="${2*base_length}" w="${2*base_width}" h="${2*base_height}" xyz="0 0 ${base_height / 2.0}" rpy="0 0 0"/>
     </link>
+    <xacro:macro name="wheel_link" params="prefix">
+        <link name="${prefix}_wheel_link">
+            <visual>
+                <geometry>
+                    <cylinder radius="${wheel_radius}" length="${wheel_length}"/>
+                </geometry>
+                <origin xyz="0 0 0" rpy="1.5708 0 0"/> <!-- pi/2 ≈ 1.5708 -->
+                <material name="grey"/>
+            </visual>
+            <collision>
+                <geometry>
+                    <cylinder radius="${wheel_radius}" length="${wheel_length}"/>
+                </geometry>
+                <origin xyz="0 0 0" rpy="1.5708 0 0"/> <!-- pi/2 ≈ 1.5708 -->
+            </collision>
+            <xacro:wheel_inertia m = "1.0" r = "${2*wheel_radius}" h = "${2*wheel_length}" xyz="0 0 0" rpy="1.5708 0 0"/>
+        </link>
+    </xacro:macro>
     <link name="caster_wheel_link">
         <visual>
@@ -44,5 +62,5 @@
             <origin xyz="0 0 0" rpy="0 0 0"/>
         </collision>
-        <xacro:sphere_inertia m="1.0" r="${wheel_radius / 2.0}" xyz="0 0 0" rpy="0 0 0"/>
+        <xacro:sphere_inertia m="1.0" r="${2*wheel_radius / 2.0}" xyz="0 0 0" rpy="0 0 0"/>
     </link>
     <xacro:wheel_link prefix="right" />

File: install/my_robot_description/share/my_robot_description/urdf/my_robot.urdf.xacro (robot description, xacro)
@@ -2,4 +2,6 @@
 <robot name="my_robot" xmlns:xacro="http://www.ros.org/wiki/xacro">
     <xacro:include filename = "/home/tayya/robot_ws/src/my_robot_description/urdf/common_properties.xacro" />
-    <xacro:include filename ="/home/tayya/robot_ws/src/my_robot_description/urdf/mobile_base.xacro"/>
+    <xacro:include filename = "/home/tayya/robot_ws/src/my_robot_description/urdf/mobile_base.xacro"/>
+    <xacro:include filename = "/home/tayya/robot_ws/src/my_robot_description/urdf/mobile_base_gazebo.xacro"/>
+    <xacro:include filename = "/home/tayya/robot_ws/src/my_robot_description/urdf/camera.xacro"/>
 </robot>
