Commit message: a

File: install/my_robot_description/share/my_robot_description/urdf/mobile_base.xacro (robot description, xacro)
@@ -12,4 +12,10 @@
     <material name="grey">
         <color rgba="0.5 0.5 0.5 1"/>
+    </material>
+    <material name = "orange">
+        <color rgba="1.0 0.5 0 1" />
+    </material>
+    <material name = "yellow">
+        <color rgba="1.0 1.0 0 1" />
     </material>
     <link name="base_footprint"/>

File: src/my_robot_description/urdf/my_robot.urdf.xacro (robot description, xacro)
@@ -5,3 +5,5 @@
     <xacro:include filename = "/home/tayya/robot_ws/src/my_robot_description/urdf/mobile_base_gazebo.xacro"/>
     <xacro:include filename = "/home/tayya/robot_ws/src/my_robot_description/urdf/camera.xacro"/>
+    <xacro:include filename = "/home/tayya/robot_ws/src/my_robot_description/urdf/arm.xacro">
+    <xacro:include filename = "/home/tayya/robot_ws/src/my_robot_description/urdf/arm_gazebo.xacro">
 </robot>
